File: electronics/trezor_one/trezor_v1.1.brd (EAGLE design)
At the start: 50 x 26.7 mm, 46 parts, among them IC1 MCP1703T-3302E/CB, K1 USB5_USB_MICRO_MOLEX475890001, K2 SWD, Q2 8MHz, U1 STM32F205RET6, U3 DISPLAY

Commit message: Using 0603 passives, changed pushbutton
Parts:
- removed S1, S2: SWITCH-MOMENTARY-2SMD, SparkFun-Electromechanical:TACTILE_SWITCH_SMD
- added S3, S4: 147873-2, 147873-2:SW_147873-2
- added U$1: (no value), flo-libs:NEWSPLORE_LOGO_BPLACE_MID
- C1, C12, C13, C14, C15, C16, C18, C2, C20, C21, C3, C4, C6, C7, C8, C9, R10, R3, R4, R6, R7, R8: device vyber:0402 -> vyber:0603
- moved U$4 4.80 mm to (28.7, 0.91)
- moved C6 3.76 mm to (8.84, 7.01)
- moved R6 3.19 mm to (10.6, 14.1), flipped to the bottom
- moved R8 2.54 mm to (9.55, 18.3), flipped to the bottom
- moved C7 1.75 mm to (8.64, 9.75)
- moved R3 1.32 mm to (7.11, 17.5), turned to 90 degrees
- moved C19 1.32 mm to (3.56, 19.0), turned to 210 degrees
- moved MB1 1.27 mm to (11.8, 4.78)
- moved C21 1.26 mm to (27.0, 10.6)
- moved R7 1.00 mm to (5.59, 17.7)
- moved C12 0.92 mm to (14.9, 25.2)
- moved C18 0.68 mm to (47.7, 2.03)
- moved MB4 0.64 mm to (4.57, 8.23)
- moved C8 0.52 mm to (14.9, 23.7)
- moved MB3 0.52 mm to (6.20, 9.86)
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Connections:
- net +3V3: now also C1.1, C12.2, C13.2, C14.2, C16.1, C3.1, C7.2, C9.2, R6.2; no longer C1.P$1, C12.P$2, C13.P$2, C14.P$2, C16.P$1, C3.P$1, C7.P$2, C9.P$2, R6.P$2
- net +5V: now also C2.1; no longer C2.P$1
- net GND: now also C1.2, C12.1, C13.1, C14.1, C15.1, C16.2, C2.2, C20.1, C21.1, C3.2, C6.1, C7.1, C8.1, C9.1, R10.1, R8.1, S3.1, S4.1; no longer C1.P$2, C12.P$1, C13.P$1, C14.P$1, C15.P$1, C16.P$2, C2.P$2, C20.P$1, C21.P$1, C3.P$2, C6.P$1, C7.P$1, C8.P$1, C9.P$1, R10.P$1, R8.P$1, S1.3, S1.4, S2.3, S2.4
- net N$10: now also C18.1; no longer C18.P$1
- net N$11: now also C4.1; no longer C4.P$1
- net N$12: now also C18.2; no longer C18.P$2
- net N$13: now also C4.2; no longer C4.P$2
- net N$18: now also R3.1; no longer R3.P$1
- net N$19: now also S4.2; no longer S1.1, S1.2
- net N$2: now also C15.2; no longer C15.P$2
- net N$20: now also S3.2; no longer S2.1, S2.2
- net N$21: now also R7.2; no longer R7.P$2
- net N$23: now also R3.2; no longer R3.P$2
- net N$24: now also R4.2; no longer R4.P$2
- net N$27: now also R7.1, R8.2; no longer R7.P$1, R8.P$2
- net N$4: now also C8.2; no longer C8.P$2
- net N$8: now also C6.2; no longer C6.P$2
- net N$9: now also R10.2; no longer R10.P$2
- net USB_D_P: now also R4.1, R6.1; no longer R4.P$1, R6.P$1
- net XTAL1: now also C20.2; no longer C20.P$2
- net XTAL2: now also C21.2; no longer C21.P$2
Routing:
- net GND: track 218.2 -> 184.5 mm, vias 56 -> 58
- net N$23: track 15.7 -> 21.5 mm, vias 2 -> 3
- net N$26: track 22.9 -> 18.5 mm
- net N$8: track 5.99 -> 9.46 mm
- net USB_D_P: track 2.43 -> 5.69 mm, vias 0 -> 1
- net N$27: track 5.52 -> 8.34 mm, vias 0 -> 1
- net N$19: track 17.8 -> 20.1 mm, vias 2 -> 3
- net XTAL2: track 7.71 -> 9.46 mm
- net +3V3: track 101.8 -> 103.3 mm
- net N$20: track 27.9 -> 27.0 mm
- net N$24: track 7.41 -> 8.18 mm
- net N$16: track 35.9 -> 35.1 mm
- net N$10: track 5.63 -> 6.16 mm
Other:
- board text added: "v1.1 02.03.2021"
- board text removed: "BOT"
- board text removed: "TOP"
